Commit message: add kinematics control

File: 2dof/install/hexapod_gz/share/hexapod_gz/urdf/hexapod_modelling_team.xacro (robot description, xacro)
@@ -4,15 +4,17 @@
      For more information, please see http://wiki.ros.org/sw_urdf_exporter -->
 <robot xmlns:xacro="http://www.ros.org/wiki/xacro"
-  name="hexapod_modelling_team">
+  name="hexapod_gz">
   <!-- Xacro defaults -->
-  <xacro:property name="mesh_dir" value="package://hexapod_modelling_team/meshes"/>
-  <!-- You can override e.g., ros2 run xacro xacro hexapod_modelling_team.xacro mesh_dir:=package://my_pkg/meshes -->
-  <!-- Import ROS2 Control -->
-  <xacro:arg name="use_sim" default="true"/>
-  <!-- Include ros2_control configuration from this package -->
-  <xacro:include filename="$(find hexapod_gz)/urdf/control.xacro" />
-  <!-- Use the ros2_control macro (Gazebo Sim hardware by default) -->
-  <xacro:ros2_control name="HexapodSystem"/>
-     <link
+  <xacro:property name="mesh_dir" value="$(find hexapod_gz)/meshes"/>
+  <!-- You can override e.g., ros2 run xacro xacro hexapod_gz.xacro mesh_dir:=package://my_pkg/meshes -->
+  <!-- World link - fixed reference frame -->
+  <link name="world"/>
+  <!-- Fixed joint to lock base_link to world (platform) -->
+  <joint name="world_fixed" type="fixed">
+    <parent link="world"/>
+    <child link="base_link"/>
+    <origin xyz="0 0 0" rpy="0 0 0"/>
+  </joint>
+  <link
     name="base_link">
     <inertial>
@@ -36,5 +38,5 @@
       <geometry>
         <mesh
-          filename="package://hexapod_modelling_team/meshes/base_link.STL" />
+          filename="file://$(find hexapod_gz)/meshes/base_link.STL" />
       </geometry>
       <material
@@ -50,5 +52,5 @@
       <geometry>
         <mesh
-          filename="package://hexapod_modelling_team/meshes/base_link.STL" />
+          filename="file://$(find hexapod_gz)/meshes/base_link.STL" />
       </geometry>
     </collision>
@@ -76,5 +78,5 @@
       <geometry>
         <mesh
-          filename="package://hexapod_modelling_team/meshes/Link1.STL" />
+          filename="file://$(find hexapod_gz)/meshes/Link1.STL" />
       </geometry>
       <material
@@ -90,5 +92,5 @@
       <geometry>
         <mesh
-          filename="package://hexapod_modelling_team/meshes/Link1.STL" />
+          filename="file://$(find hexapod_gz)/meshes/Link1.STL" />
       </geometry>
     </collision>
@@ -130,5 +132,5 @@
       <geometry>
         <mesh
-          filename="package://hexapod_modelling_team/meshes/Link_2.STL" />
+          filename="file://$(find hexapod_gz)/meshes/Link_2.STL" />
       </geometry>
       <material
@@ -144,5 +146,5 @@
       <geometry>
         <mesh
-          filename="package://hexapod_modelling_team/meshes/Link_2.STL" />
+          filename="file://$(find hexapod_gz)/meshes/Link_2.STL" />
       </geometry>
     </collision>
@@ -162,3 +164,75 @@
     <dynamics damping="0.1" friction="0.1"/>
   </joint>
+  <!-- Gazebo-specific visual and collision for base_link -->
+  <gazebo reference="base_link">
+    <visual>
+      <geometry>
+        <box>
+          <size>0.08 0.08 0.05</size>
+        </box>
+      </geometry>
+      <material>
+        <ambient>0.2 0.2 0.8 1</ambient>
+        <diffuse>0.2 0.2 0.8 1</diffuse>
+      </material>
+    </visual>
+  </gazebo>
+  <!-- Gazebo-specific visual and collision for Link1 -->
+  <gazebo reference="Link1">
+    <visual>
+      <geometry>
+        <cylinder>
+          <radius>0.02</radius>
+          <length>0.15</length>
+        </cylinder>
+      </geometry>
+      <material>
+        <ambient>0.3 0.3 0.3 1</ambient>
+        <diffuse>0.3 0.3 0.3 1</diffuse>
+      </material>
+    </visual>
+  </gazebo>
+  <!-- Gazebo-specific visual and collision for Link_2 -->
+  <gazebo reference="Link_2">
+    <visual>
+      <geometry>
+        <cylinder>
+          <radius>0.015</radius>
+          <length>0.12</length>
+        </cylinder>
+      </geometry>
+      <material>
+        <ambient>0.8 0.2 0.2 1</ambient>
+        <diffuse>0.8 0.2 0.2 1</diffuse>
+      </material>
+    </visual>
+  </gazebo>
+  <!-- ros2_control -->
+  <ros2_control name="GazeboSystem" type="system">
+    <hardware>
+      <plugin>ign_ros2_control/IgnitionSystem</plugin>
+    </hardware>
+    <joint name="rev1">
+      <command_interface name="position">
+        <param name="min">-3.14159</param>
+        <param name="max">3.14159</param>
+      </command_interface>
+      <state_interface name="position"/>
+      <state_interface name="velocity"/>
+    </joint>
+    <joint name="rev_2">
+      <command_interface name="position">
+        <param name="min">-3.14159</param>
+        <param name="max">3.14159</param>
+      </command_interface>
+      <state_interface name="position"/>
+      <state_interface name="velocity"/>
+    </joint>
+  </ros2_control>
+  <!-- Gazebo ros2_control plugin -->
+  <gazebo>
+    <plugin filename="ign_ros2_control-system" name="ign_ros2_control::IgnitionROS2ControlPlugin">
+      <parameters>$(find hexapod_gz)/config/ros2_controllers.yaml</parameters>
+    </plugin>
+  </gazebo>
 </robot>

Commit message: add sinusoidal and step function trajectory

File: 2dof/install/hexapod_gz/share/hexapod_gz/urdf/hexapod_modelling_team.xacro (robot description, xacro)
@@ -98,5 +98,5 @@
   <joint
     name="rev1"
-    type="continuous">
+    type="revolute">
     <origin
       xyz="0 0 0.0542"
@@ -108,4 +108,5 @@
     <axis
       xyz="0 0 1" />
+    <limit lower="0.0" upper="6.28" effort="10.0" velocity="10.0"/>
     <dynamics damping="0.1" friction="0.1"/>
   </joint>
@@ -152,5 +153,5 @@
   <joint
     name="rev_2"
-    type="continuous">
+    type="revolute">
     <origin
       xyz="-0.079154 0.062411 0.0045"
@@ -162,4 +163,5 @@
     <axis
       xyz="0 0 1" />
+    <limit lower="-1.47" upper="3.0" effort="10.0" velocity="10.0"/>
     <dynamics damping="0.1" friction="0.1"/>
   </joint>
@@ -214,18 +216,20 @@
     </hardware>
     <joint name="rev1">
-      <command_interface name="position">
-        <param name="min">-3.14159</param>
-        <param name="max">3.14159</param>
+      <command_interface name="effort">
+        <param name="min">-10.0</param>
+        <param name="max">10.0</param>
       </command_interface>
       <state_interface name="position"/>
       <state_interface name="velocity"/>
+      <state_interface name="effort"/>
     </joint>
     <joint name="rev_2">
-      <command_interface name="position">
-        <param name="min">-3.14159</param>
-        <param name="max">3.14159</param>
+      <command_interface name="effort">
+        <param name="min">-10.0</param>
+        <param name="max">10.0</param>
       </command_interface>
       <state_interface name="position"/>
       <state_interface name="velocity"/>
+      <state_interface name="effort"/>
     </joint>
   </ros2_control>

Commit message: add angular controller

File: 2dof/install/hexapod_gz/share/hexapod_gz/urdf/hexapod_modelling_team.xacro (robot description, xacro)
@@ -109,5 +109,5 @@
       xyz="0 0 1" />
     <limit lower="0.0" upper="6.28" effort="10.0" velocity="10.0"/>
-    <dynamics damping="0.1" friction="0.1"/>
+    <dynamics damping="0.07" friction="0.1"/>
   </joint>
   <link
@@ -164,5 +164,5 @@
       xyz="0 0 1" />
     <limit lower="-1.47" upper="3.0" effort="10.0" velocity="10.0"/>
-    <dynamics damping="0.1" friction="0.1"/>
+    <dynamics damping="0.07" friction="0.1"/>
   </joint>
   <!-- Gazebo-specific visual and collision for base_link -->
