Commit message: fix urdf file

File: 2dof/install/experiment_kit/share/experiment_kit/urdf/hexapod_modelling_team.xacro (robot description, xacro)
@@ -4,8 +4,8 @@
      For more information, please see http://wiki.ros.org/sw_urdf_exporter -->
 <robot xmlns:xacro="http://www.ros.org/wiki/xacro"
-  name="experiment_kit">
+  name="hexapod_gz">
   <!-- Xacro defaults -->
-  <xacro:property name="mesh_dir" value="$(find experiment_kit)/meshes"/>
-  <!-- You can override e.g., ros2 run xacro xacro experiment_kit.xacro mesh_dir:=package://my_pkg/meshes -->
+  <xacro:property name="mesh_dir" value="$(find hexapod_gz)/meshes"/>
+  <!-- You can override e.g., ros2 run xacro xacro hexapod_gz.xacro mesh_dir:=package://my_pkg/meshes -->
   <!-- World link - fixed reference frame -->
   <link name="world"/>
@@ -38,5 +38,5 @@
       <geometry>
         <mesh
-          filename="file://$(find experiment_kit)/meshes/base_link.STL" />
+          filename="file://$(find hexapod_gz)/meshes/base_link.STL" />
       </geometry>
       <material
@@ -52,5 +52,5 @@
       <geometry>
         <mesh
-          filename="file://$(find experiment_kit)/meshes/base_link.STL" />
+          filename="file://$(find hexapod_gz)/meshes/base_link.STL" />
       </geometry>
     </collision>
@@ -78,5 +78,5 @@
       <geometry>
         <mesh
-          filename="file://$(find experiment_kit)/meshes/Link1.STL" />
+          filename="file://$(find hexapod_gz)/meshes/Link1.STL" />
       </geometry>
       <material
@@ -92,5 +92,5 @@
       <geometry>
         <mesh
-          filename="file://$(find experiment_kit)/meshes/Link1.STL" />
+          filename="file://$(find hexapod_gz)/meshes/Link1.STL" />
       </geometry>
     </collision>
@@ -213,5 +213,5 @@
   <ros2_control name="GazeboSystem" type="system">
     <hardware>
-      <plugin>ign_ros2_control/IgnitionSystem</plugin>
+      <plugin>gz_ros2_control/GazeboSimSystem</plugin>
     </hardware>
     <joint name="rev1">
@@ -236,6 +236,6 @@
   <!-- Gazebo ros2_control plugin -->
   <gazebo>
-    <plugin filename="ign_ros2_control-system" name="ign_ros2_control::IgnitionROS2ControlPlugin">
-      <parameters>$(find experiment_kit)/config/ros2_controllers.yaml</parameters>
+    <plugin filename="gz_ros2_control-system" name="gz_ros2_control::GazeboSimROS2ControlPlugin">
+      <parameters>$(find hexapod_gz)/config/ros2_controllers.yaml</parameters>
     </plugin>
   </gazebo>
